File: Hardware/Qwiic Proximity Sensor - VCNL4040.sch (EAGLE design)
At the start: 24 parts, among them J2 SMD, J3 PTH, J4 SMD, U2 VCNL4040

Commit message: File rename
Other:
- note added: "VCNL4040 IR Proximity Sensor"
- note removed: "VCNL4040 IR Distance Sensor"
Changed lines of the file:
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@@
 <?xml version="1.0" encoding="utf-8"?>
 <!DOCTYPE eagle SYSTEM "eagle.dtd">
-<eagle version="7.7.0">
+<eagle version="9.0.0">
 <drawing>
 <settings>
 <setting alwaysvectorfont="yes"/>
+<setting keepoldvectorfont="yes"/>
 <setting verticaltext="up"/>
 </settings>
@@
 pull-up from INT</text>
 <text x="41.148" y="126.746" size="1.778" layer="97">Power</text>
-<text x="82.042" y="174.752" size="3.048" layer="97">VCNL4040 IR Distance Sensor</text>
+<text x="82.042" y="174.752" size="3.048" layer="97">VCNL4040 IR Proximity Sensor</text>
 </plain>
 <instances>
